File: PCB_Scroller/Scroller1/Scroller1.kicad_sch (KiCad schematic)
At the start: 68 parts

Commit message: Updates
Not sure if the ESP32 works...
Parts:
- removed MHole_5, MHole_6: M3, MountingHole:MountingHole_3.2mm_M3, symbol Mechanical:MountingHole
- added Mnt1: -, MT6701:BLDC Mount, symbol Mechanical:MountingHole
- D1: footprint Diode_SMD:D_MiniMELF -> Diode_SMD:D_SOD-523
Changed lines of the file:
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@@
     (stroke (width 0) (type default) (color 0 0 0 0))
   )
-  (polyline (pts (xy 226.06 48.26) (xy 226.06 60.96))
+  (polyline (pts (xy 226.06 48.26) (xy 226.06 55.88))
     (stroke (width 0) (type default) (color 0 0 0 0))
   )
@@
     (stroke (width 0) (type default) (color 0 0 0 0))
   )
-  (polyline (pts (xy 226.06 60.96) (xy 279.4 60.96))
+  (polyline (pts (xy 226.06 55.88) (xy 279.4 55.88))
     (stroke (width 0) (type default) (color 0 0 0 0))
   )
@@
     (stroke (width 0) (type default) (color 0 0 0 0))
   )
-  (polyline (pts (xy 279.4 48.26) (xy 279.4 60.96))
+  (polyline (pts (xy 279.4 48.26) (xy 279.4 55.88))
     (stroke (width 0) (type default) (color 0 0 0 0))
   )
@@
     (effects (font (size 1.27 1.27)) (justify left bottom))
   )
-  (label "WH_In" (at 36.83 132.08 0)
-    (effects (font (size 1.27 1.27)) (justify left bottom))
-  )
-  (label "WL_In" (at 36.83 134.62 0)
-    (effects (font (size 1.27 1.27)) (justify left bottom))
-  )
-  (label "VH_In" (at 36.83 127 0)
+  (label "WH_In" (at 30.48 69.85 0)
+    (effects (font (size 1.27 1.27)) (justify left bottom))
+  )
+  (label "WL_In" (at 30.48 67.31 0)
+    (effects (font (size 1.27 1.27)) (justify left bottom))
+  )
+  (label "VH_In" (at 31.75 74.93 0)
     (effects (font (size 1.27 1.27)) (justify left bottom))
   )
@@
     (effects (font (size 1.27 1.27)) (justify left bottom))
   )
-  (label "UH_In" (at 36.83 121.92 0)
-    (effects (font (size 1.27 1.27)) (justify left bottom))
-  )
-  (label "UL_In" (at 36.83 124.46 0)
-    (effects (font (size 1.27 1.27)) (justify left bottom))
-  )
-  (label "VL_In" (at 36.83 129.54 0)
+  (label "UH_In" (at 33.02 80.01 0)
+    (effects (font (size 1.27 1.27)) (justify left bottom))
+  )
+  (label "UL_In" (at 33.02 77.47 0)
+    (effects (font (size 1.27 1.27)) (justify left bottom))
+  )
+  (label "VL_In" (at 31.75 72.39 0)
     (effects (font (size 1.27 1.27)) (justify left bottom))
   )
@@
     (pin "2")
   )
-  (symbol (lib_id "Mechanical:MountingHole") (at 228.6 57.15 0) (unit 1)
-    (in_bom yes) (on_board yes) (fields_autoplaced)
-    (property "Reference" "MHole_5" (id 0) (at 231.14 55.8799 0)
-      (effects (font (size 1.27 1.27)) (justify left))
-    )
-    (property "Value" "M3" (id 1) (at 231.14 58.4199 0)
-      (effects (font (size 1.27 1.27)) (justify left))
-    )
-    (property "Footprint" "MountingHole:MountingHole_3.2mm_M3" (id 2) (at 228.6 57.15 0)
-      (effects (font (size 1.27 1.27)) hide)
-    )
-    (property "Datasheet" "~" (id 3) (at 228.6 57.15 0)
-      (effects (font (size 1.27 1.27)) hide)
-    )
-  )
   (symbol (lib_id "Switch:SW_SPST") (at 222.25 87.63 0) (unit 1)
     (in_bom yes) (on_board yes) (fields_autoplaced)
@@
     (pin "2")
   )
-  (symbol (lib_id "Mechanical:MountingHole") (at 242.57 57.15 0) (unit 1)
-    (in_bom yes) (on_board yes) (fields_autoplaced)
-    (property "Reference" "MHole_6" (id 0) (at 245.11 55.8799 0)
-      (effects (font (size 1.27 1.27)) (justify left))
-    )
-    (property "Value" "M3" (id 1) (at 245.11 58.4199 0)
-      (effects (font (size 1.27 1.27)) (justify left))
-    )
-    (property "Footprint" "MountingHole:MountingHole_3.2mm_M3" (id 2) (at 242.57 57.15 0)
-      (effects (font (size 1.27 1.27)) hide)
-    )
-    (property "Datasheet" "~" (id 3) (at 242.57 57.15 0)
-      (effects (font (size 1.27 1.27)) hide)
-    )
-  )
   (symbol (lib_id "Diode:1N4148") (at 232.41 91.44 90) (unit 1)
     (in_bom yes) (on_board yes) (fields_autoplaced)
@@
       (effects (font (size 1.27 1.27)) (justify left))
     )
-    (property "Footprint" "Diode_SMD:D_MiniMELF" (id 2) (at 107.315 167.64 0)
+    (property "Footprint" "Diode_SMD:D_SOD-523" (id 2) (at 107.315 167.64 0)
       (effects (font (size 1.27 1.27)) hide)
     )
@@
     )
     (property "Datasheet" "~" (id 3) (at 255.27 24.13 0)
+      (effects (font (size 1.27 1.27)) hide)
+    )
+  )
+  (symbol (lib_id "Mechanical:MountingHole") (at 267.97 39.37 0) (unit 1)
+    (in_bom yes) (on_board yes) (fields_autoplaced)
+    (property "Reference" "Mnt1" (id 0) (at 270.51 38.0999 0)
+      (effects (font (size 1.27 1.27)) (justify left))
+    )
+    (property "Value" "-" (id 1) (at 270.51 40.6399 0)
+      (effects (font (size 1.27 1.27)) (justify left))
+    )
+    (property "Footprint" "MT6701:BLDC Mount" (id 2) (at 267.97 39.37 0)
+      (effects (font (size 1.27 1.27)) hide)
+    )
+    (property "Datasheet" "~" (id 3) (at 267.97 39.37 0)
       (effects (font (size 1.27 1.27)) hide)
     )
@@
     )
     (path "/b70408a7-a1f3-40ab-8c1c-f15e10e04f5e"
-      (reference "D1") (unit 1) (value "ZMDxx") (footprint "Diode_SMD:D_MiniMELF")
+      (reference "D1") (unit 1) (value "ZMDxx") (footprint "Diode_SMD:D_SOD-523")
     )
     (path "/f1e68960-207d-4e96-a8e8-726eb38fb62b"
@@
       (reference "MHole_4") (unit 1) (value "M3") (footprint "MountingHole:MountingHole_3.2mm_M3")
     )
-    (path "/488d14a4-542e-41f6-bde8-b10693cdb476"
-      (reference "MHole_5") (unit 1) (value "M3") (footprint "MountingHole:MountingHole_3.2mm_M3")
-    )
-    (path "/b3c3a579-4782-4078-a553-67385e4e143c"
-      (reference "MHole_6") (unit 1) (value "M3") (footprint "MountingHole:MountingHole_3.2mm_M3")
+    (path "/cc62e911-5a16-417f-a72d-79e78a112087"
+      (reference "Mnt1") (unit 1) (value "-") (footprint "MT6701:BLDC Mount")
     )
     (path "/7f5ca6c0-eb43-425c-b2ed-6691bdb95fa6"

Commit message: Update 040523
Changed lots of things
Parts:
- UVW1: footprint Connector_FFC-FPC:Molex_200528-0060_1x06-1MP_P1.00mm_Horizontal -> Connector_FFC-FPC:Hirose_FH12-6S-0.5SH_1x06-1MP_P0.50mm_Horizontal
Changed lines of the file:
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@@
     (property "Reference" "UVW1" (id 0) (at 86.36 147.32 90))
     (property "Value" "FPC-6P" (id 1) (at 86.36 149.86 90))
-    (property "Footprint" "Connector_FFC-FPC:Molex_200528-0060_1x06-1MP_P1.00mm_Horizontal" (id 2) (at 87.63 144.78 0)
+    (property "Footprint" "Connector_FFC-FPC:Hirose_FH12-6S-0.5SH_1x06-1MP_P0.50mm_Horizontal" (id 2) (at 87.63 144.78 0)
       (effects (font (size 1.27 1.27)) hide)
     )
@@
     )
     (path "/6230ef9e-c196-4053-920d-589831945a82"
-      (reference "UVW1") (unit 1) (value "FPC-6P") (footprint "Connector_FFC-FPC:Molex_200528-0060_1x06-1MP_P1.00mm_Horizontal")
-    )
-  )
+      (reference "UVW1") (unit 1) (value "FPC-6P") (footprint "Connector_FFC-FPC:Hirose_FH12-6S-0.5SH_1x06-1MP_P0.50mm_Horizontal")
+    )
+  )
